File: light_distribution.kicad_pcb (KiCad board)
At the start: 2 copper layers, 58.4 x 43.2 mm, 12 parts, among them J1 TE_Faston_20-16AWG_Straight_T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, J2 TE_Faston_20-16AWG_Straight_T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, J3 TE_Faston_20-16AWG_Straight_T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, J4 TE_Faston_20-16AWG_Straight_T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, J5 TE_Faston_20-16AWG_Straight_T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, J6 TE_Faston_20-16AWG_Straight_T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, J7 TE_Faston_20-16AWG_Straight_T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, J8 TE_Faston_20-16AWG_Straight_T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

Commit message: migrate to project library
Parts:
- J1, J2, J3, J4, J5, J6, J7, J8: footprint Connector_Faston:TE_Faston_20-16AWG_Straight_Tab -> Toadly:TE_Faston_20-16AWG_Straight_Tab
