File: light_distribution.kicad_sch (KiCad schematic)
At the start: 8 parts, among them J1 TE_Faston_20-16AWG_Straight_T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, J2 TE_Faston_20-16AWG_Straight_T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, J3 TE_Faston_20-16AWG_Straight_T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, J4 TE_Faston_20-16AWG_Straight_T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, J5 TE_Faston_20-16AWG_Straight_T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, J6 TE_Faston_20-16AWG_Straight_T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, J7 TE_Faston_20-16AWG_Straight_T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, J8 TE_Faston_20-16AWG_Straight_T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

Commit message: export rev A
Parts:
- added H1, H2, H3, H4: MountingHole, MountingHole:MountingHole_3.5mm, symbol Mechanical:MountingHole
Changed lines of the file:
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@@
     (stroke (width 0) (type default) (color 0 0 0 0))
   )
+  (symbol (lib_id "Mechanical:MountingHole") (at 25.4 27.94 0) (unit 1)
+    (in_bom yes) (on_board yes) (fields_autoplaced)
+    (property "Reference" "H2" (id 0) (at 27.94 26.6699 0)
+      (effects (font (size 1.27 1.27)) (justify left))
+    )
+    (property "Value" "MountingHole" (id 1) (at 27.94 29.2099 0)
+      (effects (font (size 1.27 1.27)) (justify left))
+    )
+    (property "Footprint" "MountingHole:MountingHole_3.5mm" (id 2) (at 25.4 27.94 0)
+      (effects (font (size 1.27 1.27)) hide)
+    )
+    (property "Datasheet" "~" (id 3) (at 25.4 27.94 0)
+      (effects (font (size 1.27 1.27)) hide)
+    )
+  )
   (symbol (lib_id "Connector_Faston:TE_Faston_20-16AWG_Straight_Tab") (at 156.21 124.46 0) (unit 1)
     (in_bom yes) (on_board yes) (fields_autoplaced)
@@
     (pin "1")
     (pin "2")
+  )
+  (symbol (lib_id "Mechanical:MountingHole") (at 25.4 22.86 0) (unit 1)
+    (in_bom yes) (on_board yes) (fields_autoplaced)
+    (property "Reference" "H1" (id 0) (at 27.94 21.5899 0)
+      (effects (font (size 1.27 1.27)) (justify left))
+    )
+    (property "Value" "MountingHole" (id 1) (at 27.94 24.1299 0)
+      (effects (font (size 1.27 1.27)) (justify left))
+    )
+    (property "Footprint" "MountingHole:MountingHole_3.5mm" (id 2) (at 25.4 22.86 0)
+      (effects (font (size 1.27 1.27)) hide)
+    )
+    (property "Datasheet" "~" (id 3) (at 25.4 22.86 0)
+      (effects (font (size 1.27 1.27)) hide)
+    )
   )
   (symbol (lib_id "Connector_Faston:TE_Faston_20-16AWG_Straight_Tab") (at 156.21 97.79 0) (unit 1)
@@
     (pin "2")
   )
+  (symbol (lib_id "Mechanical:MountingHole") (at 25.4 33.02 0) (unit 1)
+    (in_bom yes) (on_board yes) (fields_autoplaced)
+    (property "Reference" "H3" (id 0) (at 27.94 31.7499 0)
+      (effects (font (size 1.27 1.27)) (justify left))
+    )
+    (property "Value" "MountingHole" (id 1) (at 27.94 34.2899 0)
+      (effects (font (size 1.27 1.27)) (justify left))
+    )
+    (property "Footprint" "MountingHole:MountingHole_3.5mm" (id 2) (at 25.4 33.02 0)
+      (effects (font (size 1.27 1.27)) hide)
+    )
+    (property "Datasheet" "~" (id 3) (at 25.4 33.02 0)
+      (effects (font (size 1.27 1.27)) hide)
+    )
+  )
   (symbol (lib_id "Connector_Faston:TE_Faston_20-16AWG_Straight_Tab") (at 156.21 88.9 0) (unit 1)
     (in_bom yes) (on_board yes) (fields_autoplaced)
@@
     (pin "1")
     (pin "2")
+  )
+  (symbol (lib_id "Mechanical:MountingHole") (at 25.4 38.1 0) (unit 1)
+    (in_bom yes) (on_board yes) (fields_autoplaced)
+    (property "Reference" "H4" (id 0) (at 27.94 36.8299 0)
+      (effects (font (size 1.27 1.27)) (justify left))
+    )
+    (property "Value" "MountingHole" (id 1) (at 27.94 39.3699 0)
+      (effects (font (size 1.27 1.27)) (justify left))
+    )
+    (property "Footprint" "MountingHole:MountingHole_3.5mm" (id 2) (at 25.4 38.1 0)
+      (effects (font (size 1.27 1.27)) hide)
+    )
+    (property "Datasheet" "~" (id 3) (at 25.4 38.1 0)
+      (effects (font (size 1.27 1.27)) hide)
+    )
   )
   (symbol (lib_id "Connector_Faston:TE_Faston_20-16AWG_Straight_Tab") (at 156.21 115.57 0) (unit 1)
@@
   )
   (symbol_instances
+    (path "/9576e057-8341-44b4-aa99-b8e245439c48"
+      (reference "H1") (unit 1) (value "MountingHole") (footprint "MountingHole:MountingHole_3.5mm")
+    )
+    (path "/142f7e2d-d321-4989-8327-4632df53afd6"
+      (reference "H2") (unit 1) (value "MountingHole") (footprint "MountingHole:MountingHole_3.5mm")
+    )
+    (path "/bb6dc2f3-f830-4dbe-94b1-9555bbb8201f"
+      (reference "H3") (unit 1) (value "MountingHole") (footprint "MountingHole:MountingHole_3.5mm")
+    )
+    (path "/d5c98f8b-fde2-454d-8965-dd4ac23dc191"
+      (reference "H4") (unit 1) (value "MountingHole") (footprint "MountingHole:MountingHole_3.5mm")
+    )
     (path "/a9c605ea-043e-42f5-a050-c3d6a02d4648"
       (reference "J1") (unit 1) (value "TE_Faston_20-16AWG_Straight_Tab") (footprint "TE_Faston_20-16AWG_Straight_Tab")

Commit message: migrate to project library
Parts:
- J1, J2, J3, J4, J5, J6, J7, J8: symbol Connector_Faston:TE_Faston_20-16AWG_Straight_Tab -> Toadly:TE_Faston_20-16AWG_Straight_Tab
Changed lines of the file:
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@@
     )
   )
-  (symbol (lib_id "Connector_Faston:TE_Faston_20-16AWG_Straight_Tab") (at 156.21 124.46 0) (unit 1)
+  (symbol (lib_id "Toadly:TE_Faston_20-16AWG_Straight_Tab") (at 156.21 124.46 0) (unit 1)
     (in_bom yes) (on_board yes) (fields_autoplaced)
     (property "Reference" "J8" (id 0) (at 161.29 124.4599 0)
@@
     )
   )
-  (symbol (lib_id "Connector_Faston:TE_Faston_20-16AWG_Straight_Tab") (at 156.21 97.79 0) (unit 1)
+  (symbol (lib_id "Toadly:TE_Faston_20-16AWG_Straight_Tab") (at 156.21 97.79 0) (unit 1)
     (in_bom yes) (on_board yes) (fields_autoplaced)
     (property "Reference" "J5" (id 0) (at 161.29 97.7899 0)
@@
     (pin "2")
   )
-  (symbol (lib_id "Connector_Faston:TE_Faston_20-16AWG_Straight_Tab") (at 156.21 71.12 0) (unit 1)
+  (symbol (lib_id "Toadly:TE_Faston_20-16AWG_Straight_Tab") (at 156.21 71.12 0) (unit 1)
     (in_bom yes) (on_board yes) (fields_autoplaced)
     (property "Reference" "J2" (id 0) (at 161.29 71.1199 0)
@@
     (pin "2")
   )
-  (symbol (lib_id "Connector_Faston:TE_Faston_20-16AWG_Straight_Tab") (at 118.11 71.12 180) (unit 1)
+  (symbol (lib_id "Toadly:TE_Faston_20-16AWG_Straight_Tab") (at 118.11 71.12 180) (unit 1)
     (in_bom yes) (on_board yes) (fields_autoplaced)
     (property "Reference" "J1" (id 0) (at 117.475 66.04 0))
@@
     (pin "2")
   )
-  (symbol (lib_id "Connector_Faston:TE_Faston_20-16AWG_Straight_Tab") (at 156.21 106.68 0) (unit 1)
+  (symbol (lib_id "Toadly:TE_Faston_20-16AWG_Straight_Tab") (at 156.21 106.68 0) (unit 1)
     (in_bom yes) (on_board yes) (fields_autoplaced)
     (property "Reference" "J6" (id 0) (at 161.29 106.6799 0)
@@
     )
   )
-  (symbol (lib_id "Connector_Faston:TE_Faston_20-16AWG_Straight_Tab") (at 156.21 88.9 0) (unit 1)
+  (symbol (lib_id "Toadly:TE_Faston_20-16AWG_Straight_Tab") (at 156.21 88.9 0) (unit 1)
     (in_bom yes) (on_board yes) (fields_autoplaced)
     (property "Reference" "J4" (id 0) (at 161.29 88.8999 0)
@@
     )
   )
-  (symbol (lib_id "Connector_Faston:TE_Faston_20-16AWG_Straight_Tab") (at 156.21 115.57 0) (unit 1)
+  (symbol (lib_id "Toadly:TE_Faston_20-16AWG_Straight_Tab") (at 156.21 115.57 0) (unit 1)
     (in_bom yes) (on_board yes) (fields_autoplaced)
     (property "Reference" "J7" (id 0) (at 161.29 115.5699 0)
@@
     (pin "2")
   )
-  (symbol (lib_id "Connector_Faston:TE_Faston_20-16AWG_Straight_Tab") (at 156.21 80.01 0) (unit 1)
+  (symbol (lib_id "Toadly:TE_Faston_20-16AWG_Straight_Tab") (at 156.21 80.01 0) (unit 1)
     (in_bom yes) (on_board yes) (fields_autoplaced)
     (property "Reference" "J3" (id 0) (at 161.29 80.0099 0)
